File: KICAD/ZED_F9P_minimal_design/ZED_F9P_minimal/ZED_F9P_minimal.kicad_sch (KiCad schematic)
At the start: 3 parts, among them IC1 ZED-F9P-15B

Commit message: PCB
Parts:
- removed AE1: Antenna, symbol Device:Antenna
- C1: footprint (none) -> Capacitor_SMD:C_0201_0603Metric
- IC1: footprint ZEDF9P15B -> RF_GPS:ublox_ZED
Connections:
- net Antenna: now reaches IC1.2 (RF_IN)
Changed lines of the file:
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@@
 		)
 	)
-	(symbol
-		(lib_id "Device:Antenna")
-		(at 73.66 20.32 0)
-		(unit 1)
-		(exclude_from_sim no)
-		(in_bom yes)
-		(on_board yes)
-		(dnp no)
-		(fields_autoplaced yes)
-		(property "Reference" "AE1"
-			(at 76.2 19.6849 0)
-			(effects
-				(font
-					(size 1.27 1.27)
-				)
-				(justify left)
-			)
-		)
-		(property "Value" "Antenna"
-			(at 76.2 22.2249 0)
-			(effects
-				(font
-					(size 1.27 1.27)
-				)
-				(justify left)
-			)
-		)
-		(property "Footprint" ""
-			(at 73.66 20.32 0)
-			(effects
-				(font
-					(size 1.27 1.27)
-				)
-				(hide yes)
-			)
-		)
-		(property "Datasheet" "~"
-			(at 73.66 20.32 0)
-			(effects
-				(font
-					(size 1.27 1.27)
-				)
-				(hide yes)
-			)
-		)
-		(property "Description" "Antenna"
-			(at 73.66 20.32 0)
-			(effects
-				(font
-					(size 1.27 1.27)
-				)
-				(hide yes)
-			)
-		)
-		(pin "1"
-		)
-		(instances
-			(project ""
-				(path "/b6a75013-49e3-468e-8fb3-ec14dcddf343"
-					(reference "AE1")
-					(unit 1)
-				)
-			)
+	(hierarchical_label "Antenna"
+		(shape input)
+		(at 73.66 25.4 0)
+		(fields_autoplaced yes)
+		(effects
+			(font
+				(size 1.27 1.27)
+			)
+			(justify left)
 		)
 	)
@@
 			)
 		)
-		(property "Footprint" "ZEDF9P15B"
+		(property "Footprint" "RF_GPS:ublox_ZED"
 			(at 120.65 126.67 0)
+			(show_name yes)
 			(effects
 				(font
@@
 			)
 		)
-		(property "Footprint" ""
+		(property "Footprint" "Capacitor_SMD:C_0201_0603Metric"
 			(at 39.0652 64.77 0)
 			(effects
