File: Hardware/KICAD/ZED_F9P_minimal_design/ZED_F9P_minimal/ZED_F9P_minimal.kicad_sch (KiCad schematic)
At the start: 28 parts, among them J1 EMPCB.SMAFSTJ.B.HT, J2 DF11-18DS-2DSA06, U1 OPA2365AID, U2 LM1086IT-ADJ/NOPB, U3 ZED-F9P

Commit message: modifications
corrected critical mistakes on rf input
added power on state led
removed RF input testpoint
Parts:
- removed D3: 3.7, Diode_SMD:D_0805_2012Metric, symbol Device:D_TVS
- removed TP1: TestPoint, TestPoint:CONN1_5011_KEY, symbol Connector:TestPoint
- added D3: LED_rouge, LED_SMD:LED_0805_2012Metric, symbol Device:LED
- added R4: 330, res_SMD_330ohm:RC0805N_YAG, symbol Device:R
- U2: value LM1086IT-ADJ/NOPB -> ~
- renumbered J2 to INPUTS1, U3 to ZED-F9P1
Connections:
- net 3v3_puce: now also R4.2
- net GND: now also D3.1 (K); no longer R5.1, ZED-F9P1.20 (RTK_STAT)
- new net: D3.2 (A), R4.1
- new net: R5.1, ZED-F9P1.20 (RTK_STAT)
Other:
- moved on the sheet: D2, TP4
