File: Hardware/KICAD/ZED_F9P_minimal_design/ZED_F9P_minimal/ZED_F9P_minimal.kicad_sch (KiCad schematic)
At the start: 28 parts

Commit message: update
update
Parts:
- added D4: 3.6, Diode_SMD:SOD323_DIO, symbol Device:D_Zener
- D2: footprint Diode_SMD:D_SOD-323 -> Diode_SMD:SOD323_DIO
- L1: footprint Inductor_SMD:L_0805_2012Metric -> Inductor_SMD:IND_786110A_WRE
Connections:
- net GND: now also D4.1 (K)
- net RF_IN: now also D4.2 (A)
Changed lines of the file:
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@@
 	)
 	(junction
+		(at 96.52 40.64)
+		(diameter 0)
+		(color 0 0 0 0)
+	)
+	(junction
 		(at 62.23 83.82)
 		(diameter 0)
@@
 	)
 	(junction
+		(at 96.52 71.12)
+		(diameter 0)
+		(color 0 0 0 0)
+	)
+	(junction
 		(at 107.95 110.49)
 		(diameter 0)
@@
 	(wire
 		(pts
+			(xy 96.52 54.61) (xy 96.52 71.12)
+		)
+		(stroke
+			(width 0)
+			(type default)
+		)
+	)
+	(wire
+		(pts
 			(xy 46.99 134.62) (xy 46.99 142.24)
 		)
@@
 	(wire
 		(pts
+			(xy 96.52 71.12) (xy 100.33 71.12)
+		)
+		(stroke
+			(width 0)
+			(type default)
+		)
+	)
+	(wire
+		(pts
 			(xy 107.95 104.14) (xy 107.95 110.49)
 		)
@@
 	(wire
 		(pts
-			(xy 78.74 71.12) (xy 100.33 71.12)
+			(xy 78.74 71.12) (xy 96.52 71.12)
 		)
 		(stroke
@@
 	(wire
 		(pts
-			(xy 78.74 40.64) (xy 100.33 40.64)
+			(xy 78.74 40.64) (xy 96.52 40.64)
 		)
 		(stroke
@@
 	(wire
 		(pts
+			(xy 96.52 40.64) (xy 100.33 40.64)
+		)
+		(stroke
+			(width 0)
+			(type default)
+		)
+	)
+	(wire
+		(pts
 			(xy 168.91 52.07) (xy 168.91 64.77)
 		)
@@
 	(wire
 		(pts
+			(xy 96.52 46.99) (xy 96.52 40.64)
+		)
+		(stroke
+			(width 0)
+			(type default)
+		)
+	)
+	(wire
+		(pts
 			(xy 115.57 104.14) (xy 116.84 104.14)
 		)
@@
 	)
 	(symbol
+		(lib_id "Device:D_Zener")
+		(at 96.52 50.8 90)
+		(unit 1)
+		(exclude_from_sim no)
+		(in_bom yes)
+		(on_board yes)
+		(dnp no)
+		(property "Reference" "D4"
+			(at 94.234 50.8 90)
+			(effects
+				(font
+					(size 1.27 1.27)
+				)
+				(justify left)
+			)
+		)
+		(property "Value" "3.6"
+			(at 94.488 49.53 90)
+			(effects
+				(font
+					(size 1.27 1.27)
+				)
+				(justify left)
+			)
+		)
+		(property "Footprint" "Diode_SMD:SOD323_DIO"
+			(at 96.52 50.8 0)
+			(effects
+				(font
+					(size 1.27 1.27)
+				)
+				(hide yes)
+			)
+		)
+		(property "Datasheet" "~"
+			(at 96.52 50.8 0)
+			(effects
+				(font
+					(size 1.27 1.27)
+				)
+				(hide yes)
+			)
+		)
+		(property "Description" "Zener diode"
+			(at 96.52 50.8 0)
+			(effects
+				(font
+					(size 1.27 1.27)
+				)
+				(hide yes)
+			)
+		)
+		(property "Height" ""
+			(at 96.52 50.8 0)
+			(effects
+				(font
+					(size 1.27 1.27)
+				)
+				(hide yes)
+			)
+		)
+		(property "Manufacturer_Name" ""
+			(at 96.52 50.8 0)
+			(effects
+				(font
+					(size 1.27 1.27)
+				)
+				(hide yes)
+			)
+		)
+		(property "Manufacturer_Part_Number" ""
+			(at 96.52 50.8 0)
+			(effects
+				(font
+					(size 1.27 1.27)
+				)
+				(hide yes)
+			)
+		)
+		(property "Mouser Part Number" ""
+			(at 96.52 50.8 0)
+			(effects
+				(font
+					(size 1.27 1.27)
+				)
+				(hide yes)
+			)
+		)
+		(property "Mouser Price/Stock" ""
+			(at 96.52 50.8 0)
+			(effects
+				(font
+					(size 1.27 1.27)
+				)
+				(hide yes)
+			)
+		)
+		(pin "1"
+		)
+		(pin "2"
+		)
+		(instances
+			(project "ZED_F9P_minimal"
+				(path "/b6a75013-49e3-468e-8fb3-ec14dcddf343"
+					(reference "D4")
+					(unit 1)
+				)
+			)
+		)
+	)
+	(symbol
 		(lib_id "Device:C")
 		(at 95.25 106.68 180)
@@
 			)
 		)
-		(property "Footprint" "Inductor_SMD:L_0805_2012Metric"
+		(property "Footprint" "Inductor_SMD:IND_786110A_WRE"
 			(at 78.74 46.99 0)
 			(effects
@@
 			)
 		)
-		(property "Footprint" "Diode_SMD:D_SOD-323"
+		(property "Footprint" "Diode_SMD:SOD323_DIO"
 			(at 100.33 50.8 0)
 			(effects
