File: Hardware/KICAD/ZED_F9P_minimal_design/ZED_F9P_minimal/ZED_F9P_minimal.kicad_pcb (KiCad board)
At the start: 2 copper layers, 60 x 45.5 mm, 32 parts

Commit message: update
update
Parts:
- added D4: 3.6, Diode_SMD:SOD323_DIO, F.Cu at (61.5, 28.7)
- D2: footprint Diode_SMD:D_SOD-323 -> Diode_SMD:SOD323_DIO
- L1: footprint Inductor_SMD:L_0805_2012Metric -> Inductor_SMD:IND_786110A_WRE
- moved D2 2.26 mm to (63.8, 28.6)
- moved C2 0.56 mm to (55.9, 29.1)
- moved L1 0.44 mm to (59.5, 28.3)
Connections:
- INPUTS1 pad 19: GND -> (no net)
- INPUTS1 pad 20: GND -> (no net)
Routing:
- net GND: vias 388 -> 392
