File: Hardware/KICAD/ZED_F9P_minimal_design/ZED_F9P_minimal/fab PCB/ZED_F9P_minimal.kicad_pcb (KiCad board)
At the start: 2 copper layers, 60 x 45.5 mm, 32 parts

Commit message: fab files
modifs
Parts:
- moved R1 0.83 mm to (57.6, 31.8)
- moved C2 0.47 mm to (56.8, 28.7)
Routing:
- net Net-(C2-Pad1): track 5.29 -> 4.61 mm
- net GND: vias 411 -> 407
Changed lines of the file:
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@@
 	(footprint "Capacitor_SMD:C_0805_2012Metric"
 		(layer "F.Cu")
-		(at 56.3 28.775 90)
+		(at 56.75925 28.693599 90)
 		(descr "Capacitor SMD 0805 (2012 Metric), square (rectangular) end terminal, IPC_7351 nominal, (Body size source: IPC-SM-782 page 76, https://www.pcb-3d.com/wordpress/wp-content/uploads/ipc-sm-782a_amendment_1_and_2.pdf, https://docs.google.com/spreadsheets/d/1BsfQQcO9C6DZCsRaXUlFlo91Tg2WpOkGARC1WS5S8t0/edit?usp=sharing), generated with kicad-footprint-generator")
 		(tags "capacitor")
 		(property "Reference" "C2"
-			(at 4.993599 3.8 90)
+			(at 4.993599 3.54075 90)
 			(layer "F.SilkS")
 			(effects
@@
 		(at 77.45 27.455 -90)
 		(property "Reference" "SMA1"
-			(at -4.155 10.4 0)
+			(at -3.23 11 90)
 			(layer "F.SilkS")
 			(effects
@@
 	(footprint "res_SMD_330ohm:RC0805N_YAG"
 		(layer "F.Cu")
-		(at 56.7731 31.925)
+		(at 57.59325 31.804)
 		(tags "RC0805FR-07330RL ")
 		(property "Reference" "R1"
-			(at 3.4519 -7 0)
+			(at 2.70675 -7.104 0)
 			(unlocked yes)
 			(layer "F.SilkS")
@@
 			(polygon
 				(pts
-					(xy 56.481 31.3789) (xy 57.0652 31.3789) (xy 57.0652 32.4711) (xy 56.481 32.4711)
+					(xy 57.30115 31.2579) (xy 57.88535 31.2579) (xy 57.88535 32.3501) (xy 57.30115 32.3501)
 				)
 			)
@@
 		(layer "F.SilkS")
 	)
-	(gr_poly
-		(pts
-			(xy 52.15 20.4) (xy 52.15 21.15) (xy 51.7 21.69735) (xy 43.5 21.69735) (xy 43.05 21.4) (xy 43.05 20.25)
-			(xy 43.55 19.82235) (xy 51.7 19.82235)
-		)
-		(stroke
-			(width 0)
-			(type solid)
-		)
-		(fill solid)
-		(layer "F.Mask")
-	)
-	(gr_poly
-		(pts
-			(xy 44.731137 20.309541) (xy 44.731137 21.059541) (xy 44.725 21.7) (xy 43.975 21.7) (xy 43.55 22.1)
-			(xy 41.475 22.1) (xy 41.4 21.725) (xy 43.35 19.825) (xy 44.725 19.825)
-		)
-		(stroke
-			(width 0)
-			(type solid)
-		)
-		(fill solid)
-		(layer "F.Mask")
-	)
-	(gr_poly
-		(pts
-			(xy 60 26.55) (xy 59.05 28.4) (xy 58.55 28.15) (xy 52.075 21.7) (xy 50.95 21.7) (xy 50.925 19.825)
-			(xy 52.975 19.825) (xy 59.625 26.5)
-		)
-		(stroke
-			(width 0)
-			(type solid)
-		)
-		(fill solid)
-		(layer "F.Mask")
-	)
 	(gr_rect
 		(start 75.1 24.075)
@@
 	(gr_poly
 		(pts
-			(xy 75.6 27.07765) (xy 75.6 27.87765) (xy 75.15 28.4) (xy 59.05 28.4) (xy 58.65 28.12765) (xy 58.65 26.9)
-			(xy 59 26.55) (xy 75.15 26.55)
+			(xy 75.6 27.07765) (xy 75.6 27.87765) (xy 75.15 28.4) (xy 64 28.4) (xy 63.3 27.87765) (xy 63.3 27)
+			(xy 64 26.55) (xy 75.15 26.55)
 		)
 		(stroke
@@
 	(gr_text "RTK STATUS"
 		(at 20.75 44.5 0)
-		(layer "F.SilkS" knockout)
+		(layer "Edge.Cuts")
 		(effects
 			(font
@@
 	(gr_text "PWR ON"
 		(at 27.5 44.4 0)
-		(layer "F.SilkS" knockout)
+		(layer "Edge.Cuts")
 		(effects
 			(font
@@
 	)
 	(via
-		(at 59.375 34.425)
-		(size 0.6)
-		(drill 0.3)
-		(layers "F.Cu" "B.Cu")
-		(free yes)
-		(net 2)
-	)
-	(via
 		(at 54.1 58.375)
 		(size 0.6)
@@
 	)
 	(via
-		(at 58.975 31.775)
-		(size 0.6)
-		(drill 0.3)
-		(layers "F.Cu" "B.Cu")
-		(free yes)
-		(net 2)
-	)
-	(via
 		(at 64.1 26.45)
 		(size 0.6)
@@
 	)
 	(via
-		(at 57.825 30.55)
-		(size 0.6)
-		(drill 0.3)
-		(layers "F.Cu" "B.Cu")
-		(free yes)
-		(net 2)
-	)
-	(via
 		(at 64.75 51.625)
 		(size 0.6)
@@
 	)
 	(via
-		(at 59.4 33.025)
-		(size 0.6)
-		(drill 0.3)
-		(layers "F.Cu" "B.Cu")
-		(free yes)
-		(net 2)
-	)
-	(via
 		(at 52.5 58.4)
 		(size 0.6)
@@
 	)
 	(segment
-		(start 55.925 31.925)
-		(end 55.925 30.1)
+		(start 56.74515 31.804)
+		(end 56.74515 29.657699)
 		(width 0.2)
 		(layer "F.Cu")
@@
 	)
 	(segment
-		(start 55.925 30.1)
-		(end 56.4085 29.6165)
+		(start 56.74515 29.657699)
+		(end 56.75925 29.643599)
 		(width 0.2)
 		(layer "F.Cu")
@@
 	)
 	(segment
-		(start 56.4085 29.6165)
+		(start 56.786349 29.6165)
 		(end 59.19135 29.6165)
 		(width 0.2)
@@
 	)
 	(segment
+		(start 56.75925 29.643599)
+		(end 56.786349 29.6165)
+		(width 0.2)
+		(layer "F.Cu")
+		(net 3)
+	)
+	(segment
 		(start 42 22.45)
 		(end 42 23.4)
@@
 	)
 	(segment
-		(start 58.50385 32.80765)
-		(end 57.6212 31.925)
+		(start 65.025 38.1)
+		(end 67.4 38.1)
 		(width 0.4)
 		(layer "F.Cu")
@@
 	)
 	(segment
-		(start 65.025 38.1)
-		(end 67.4 38.1)
+		(start 58.50385 35.3815)
+		(end 58.50385 31.8665)
 		(width 0.4)
 		(layer "F.Cu")
@@
 	)
 	(segment
+		(start 58.50385 31.8665)
+		(end 58.44135 31.804)
+		(width 0.4)
+		(layer "F.Cu")
+		(net 17)
+	)
+	(segment
 		(start 69.07 39.8769)
 		(end 67.8 39.8769)
@@
 		(width 0.4)
 		(layer "F.Cu")
-		(net 17)
-	)
-	(segment
-		(start 58.50385 35.3815)
-		(end 58.50385 32.80765)
-		(width 0.4)
-		(layer "F.Cu")
